File: PCB/Team18_V1.3.sch (EAGLE design)
At the start: 62 parts, among them IC1 STM32F746ZGT6, J1 5.5x2.1mm Barrel, J2 CORTEX_DEBUG_PTH, P1 1-1473005-4, U1 TPPM0110DWPRDWP20_3P81X2P79-L, X1 2520-

Commit message: pcbsleep
Parts:
- removed HIGH_FREQ_OSC: 25 MHZ, SparkFun-Clocks:CRYSTAL-26MHZSMD-3.2X2.5
- added J3: 22-27-2041-04, con-molex:22-27-2041-04
- added Q1: (no value), adafruit:CRYSTALHC49UP
Connections:
- new net SENSOR_UART: IC1.PF6, J3-2.S
- net GND: now also J3-4.S; no longer HIGH_FREQ_OSC.3
- net OSC_IN: now also Q1.1; no longer HIGH_FREQ_OSC.1
- net OSC_OUT: now also Q1.2; no longer HIGH_FREQ_OSC.2
- net VDD: now also J3-3.S
Changed lines of the file:
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@@
 <parts>
 <part name="IC1" library="477_LIBRARY" deviceset="STM32F746ZGT6" device=""/>
-<part name="HIGH_FREQ_OSC" library="SparkFun-Clocks" library_urn="urn:adsk.eagle:library:511" deviceset="CRYSTAL-26MHZ" device="SMD-3.2X2.5" package3d_urn="urn:adsk.eagle:package:37521/1" value="25 MHZ"/>
 <part name="LOW_FREQ_OSC" library="mbed-HDK-Oscillator" deviceset="GENERIC-CRYSTAL" device="_FC135"/>
 <part name="C1" library="adafruit" library_urn="urn:adsk.eagle:library:420" deviceset="C-US" device="C0805" package3d_urn="urn:adsk.eagle:package:6240337/1" value="1.2pF"/>
@@
 <part name="C42" library="rcl" library_urn="urn:adsk.eagle:library:334" deviceset="C-EU" device="C0805" package3d_urn="urn:adsk.eagle:package:23617/2" value="100nF"/>
 <part name="J2" library="SparkFun-Connectors" library_urn="urn:adsk.eagle:library:513" deviceset="CORTEX_DEBUG" device="_PTH" package3d_urn="urn:adsk.eagle:package:38290/1"/>
+<part name="Q1" library="adafruit" library_urn="urn:adsk.eagle:library:420" deviceset="CRYSTAL" device="HC49UP" package3d_urn="urn:adsk.eagle:package:6240908/1"/>
+<part name="J3" library="con-molex" library_urn="urn:adsk.eagle:library:165" deviceset="22-?-04" device="27-2041"/>
 </parts>
 <sheets>
@@
 <attribute name="VALUE" x="171.45" y="86.36" size="1.778" layer="96" align="center-left"/>
 </instance>
-<instance part="HIGH_FREQ_OSC" gate="G$1" x="-17.78" y="10.16" smashed="yes">
-<attribute name="VALUE" x="-16.256" y="8.636" size="1.778" layer="96" font="vector" align="top-left"/>
-<attribute name="NAME" x="-19.05" y="8.636" size="1.778" layer="95" font="vector" align="top-right"/>
-</instance>
 <instance part="LOW_FREQ_OSC" gate="G$1" x="-17.78" y="48.26" smashed="yes">
 <attribute name="NAME" x="-20.32" y="50.546" size="1.27" layer="95" font="vector" ratio="12"/>
@@
 <attribute name="VALUE" x="182.88" y="244.094" size="1.778" layer="96" font="vector"/>
 </instance>
+<instance part="Q1" gate="G$1" x="-17.78" y="10.16" smashed="yes">
+<attribute name="NAME" x="-15.24" y="11.176" size="1.778" layer="95"/>
+<attribute name="VALUE" x="-15.24" y="7.62" size="1.778" layer="96"/>
+</instance>
+<instance part="J3" gate="-1" x="347.98" y="259.08" smashed="yes">
+<attribute name="NAME" x="350.52" y="258.318" size="1.524" layer="95"/>
+<attribute name="VALUE" x="347.218" y="260.477" size="1.778" layer="96"/>
+</instance>
+<instance part="J3" gate="-2" x="347.98" y="254" smashed="yes">
+<attribute name="NAME" x="350.52" y="253.238" size="1.524" layer="95"/>
+</instance>
+<instance part="J3" gate="-3" x="347.98" y="248.92" smashed="yes">
+<attribute name="NAME" x="350.52" y="248.158" size="1.524" layer="95"/>
+</instance>
+<instance part="J3" gate="-4" x="347.98" y="243.84" smashed="yes">
+<attribute name="NAME" x="350.52" y="243.078" size="1.524" layer="95"/>
+</instance>
 </instances>
 <busses>
@@
 <pinref part="C3" gate="G$1" pin="1"/>
 <wire x1="-25.4" y1="5.08" x2="-25.4" y2="10.16" width="0.1524" layer="91"/>
-<pinref part="HIGH_FREQ_OSC" gate="G$1" pin="1"/>
 <wire x1="-25.4" y1="10.16" x2="-20.32" y2="10.16" width="0.1524" layer="91"/>
 <pinref part="IC1" gate="G$1" pin="PHO"/>
@@
 <junction x="-25.4" y="10.16"/>
 <label x="55.88" y="15.24" size="1.778" layer="95"/>
+<pinref part="Q1" gate="G$1" pin="1"/>
 </segment>
 </net>
 <net name="OSC_OUT" class="0">
 <segment>
-<pinref part="HIGH_FREQ_OSC" gate="G$1" pin="2"/>
 <wire x1="-15.24" y1="10.16" x2="-10.16" y2="10.16" width="0.1524" layer="91"/>
 <pinref part="C4" gate="G$1" pin="1"/>
@@
 <junction x="-10.16" y="10.16"/>
 <label x="55.88" y="12.7" size="1.778" layer="95"/>
+<pinref part="Q1" gate="G$1" pin="2"/>
 </segment>
 </net>
@@
 <segment>
 <pinref part="C3" gate="G$1" pin="2"/>
-<wire x1="-25.4" y1="-2.54" x2="-25.4" y2="-5.08" width="0.1524" layer="91"/>
 <pinref part="SUPPLY3" gate="GND" pin="GND"/>
-<pinref part="HIGH_FREQ_OSC" gate="G$1" pin="3"/>
-<wire x1="-25.4" y1="-5.08" x2="-25.4" y2="-7.62" width="0.1524" layer="91"/>
-<wire x1="-17.78" y1="5.08" x2="-17.78" y2="-5.08" width="0.1524" layer="91"/>
-<wire x1="-17.78" y1="-5.08" x2="-25.4" y2="-5.08" width="0.1524" layer="91"/>
-<junction x="-25.4" y="-5.08"/>
+<wire x1="-25.4" y1="-2.54" x2="-25.4" y2="-7.62" width="0.1524" layer="91"/>
 </segment>
 <segment>
@@
 <wire x1="162.56" y1="248.92" x2="180.34" y2="248.92" width="0.1524" layer="91"/>
 </segment>
+<segment>
+<pinref part="J3" gate="-4" pin="S"/>
+<wire x1="345.44" y1="243.84" x2="335.28" y2="243.84" width="0.1524" layer="91"/>
+<label x="335.28" y="243.84" size="1.778" layer="95"/>
+</segment>
 </net>
 <net name="OSC32_IN" class="0">
@@
 <pinref part="C42" gate="G$1" pin="1"/>
 <wire x1="180.34" y1="259.08" x2="162.56" y2="259.08" width="0.1524" layer="91"/>
+</segment>
+<segment>
+<pinref part="J3" gate="-3" pin="S"/>
+<wire x1="345.44" y1="248.92" x2="335.28" y2="248.92" width="0.1524" layer="91"/>
+<label x="335.28" y="248.92" size="1.778" layer="95"/>
 </segment>
 </net>
@@
 </segment>
 </net>
+<net name="SENSOR_UART" class="0">
+<segment>
+<pinref part="J3" gate="-2" pin="S"/>
+<wire x1="345.44" y1="254" x2="335.28" y2="254" width="0.1524" layer="91"/>
+<label x="327.66" y="254" size="1.778" layer="95"/>
+</segment>
+<segment>
+<pinref part="IC1" gate="G$1" pin="PF6"/>
+<wire x1="71.12" y1="27.94" x2="55.88" y2="27.94" width="0.1524" layer="91"/>
+<label x="48.26" y="27.94" size="1.778" layer="95"/>
+</segment>
+</net>
