File: PCB/Team18_V1.3.brd (EAGLE design)
At the start: 181.1 x 100 mm, 61 parts, among them IC1 STM32F746ZGT6, J1 5.5x2.1mm Barrel, P1 1-1473005-4, U1 TPPM0110DWPRDWP20_3P81X2P79-L, X1 2520-

Commit message: EagleAllNite
Parts:
- added C42: 100nF, rcl:C0805
- added DRILEGEND: (no value), drilegend:DRILEGEND
- moved JTAG 190.2 mm to (67.9, 96.4), turned to 180 degrees
- moved R2 76.3 mm to (-55.2, 59.8), flipped to the bottom, turned to 270 degrees
- moved C1 47.6 mm to (52.2, 40.8)
- moved C15 47.6 mm to (67.3, 55.2)
- moved C2 47.6 mm to (54.9, 40.8)
- moved C4 47.6 mm to (62.8, 41.2)
- moved C5 47.6 mm to (67.3, 59.4)
- moved C6 47.6 mm to (67.3, 63.6)
- moved LOW_FREQ_OSC 47.6 mm to (53.6, 41.9)
- moved C11 47.6 mm to (67.3, 51.1)
- moved C12 47.6 mm to (55.0, 47.9)
- moved C13 47.6 mm to (58.9, 47.9)
- moved C16 47.6 mm to (71.6, 63.6)
- moved C3 47.6 mm to (60.0, 41.2)
- moved C8 47.6 mm to (50.7, 64.5)
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Connections:
- new net KEY: JTAG.7
- net GND: now also C42.2
- net RESET: now also IC1.134, IC1.25
- net SWCLK: now also IC1.109
- net SWDIO: now also IC1.105
- net SWO: now also IC1.133
- net VDD: now also C42.1
Routing:
- net GND: track 7.70 -> 534.6 mm, vias 2 -> 25
- net 3.3V: track 0.00 -> 119.4 mm, vias 0 -> 2
- net 5VOUT: track 0.00 -> 110.9 mm, vias 0 -> 3
- net 5VIN: track 0.00 -> 107.4 mm
- net UART5_TX: track 0.00 -> 104.5 mm, vias 0 -> 2
- net UART5_RX: track 0.00 -> 104.2 mm, vias 0 -> 2
- net VDD: track 0.00 -> 80.7 mm, vias 0 -> 15
- net QSPI_CS: track 0.00 -> 75.7 mm, vias 0 -> 1
- net RESET: track 0.00 -> 54.4 mm, vias 0 -> 2
- net SWO: track 0.00 -> 53.4 mm, vias 0 -> 2
- net 1.8V: track 0.00 -> 47.1 mm, vias 0 -> 2
- net N$7: track 0.00 -> 40.2 mm
- net SWCLK: track 0.00 -> 39.6 mm
- net SWDIO: track 0.00 -> 36.7 mm
- net QIO0: track 0.00 -> 33.2 mm
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- added copper zone on layer 3, net 1.8V
- added copper zone on layer 3, net VDD

Commit message: PCB
Parts:
- removed JTAG: (no value), Wurth_Elektronik_Electromechanic_Board_to_Board_Connectors_rev18b:62201021821
- added J2: CORTEX_DEBUG_PTH, SparkFun-Connectors:2X5-PTH-1.27MM
Connections:
- new net N$19: J2.8
- net 3.3V: no longer C23.1, C24.1, C25.1, C26.1, C35.1, C37.2, P1.191, P1.192, P1.193, P1.194, R3.2, U1.4
- net GND: now also J2.3, J2.5, J2.9; no longer JTAG.3, JTAG.5, JTAG.9
- net KEY: now also J2.7; no longer JTAG.7
- net RESET: now also J2.10; no longer IC1.134, JTAG.10
- net SWCLK: now also J2.4; no longer JTAG.4
- net SWDIO: now also J2.2; no longer JTAG.2
- net SWO: now also J2.6; no longer JTAG.6
- net VDD: now also C23.1, C24.1, C25.1, C26.1, C35.1, C37.2, J2.1, P1.191, P1.192, P1.193, P1.194, R3.2, U1.4; no longer JTAG.1
Routing:
- net 3.3V: track 119.4 -> 27.3 mm, vias 2 -> 1
- net VDD: track 80.7 -> 144.3 mm, vias 15 -> 37
- net 5VOUT: track 110.9 -> 160.1 mm, vias 3 -> 19
- net 5VIN: track 107.4 -> 67.9 mm
- net RESET: track 54.4 -> 77.1 mm
- net GND: track 534.6 -> 551.9 mm, vias 25 -> 47
- net N$6: track 19.6 -> 36.5 mm
- net RUN: track 0.00 -> 9.06 mm
- net N$1: track 0.00 -> 5.60 mm, vias 0 -> 1
- net 1.8V: track 47.1 -> 51.3 mm, vias 2 -> 10
- net OSC_OUT: track 5.74 -> 9.55 mm, vias 0 -> 1
- net N$8: track 18.5 -> 15.0 mm
- net QSPICLK: track 30.8 -> 32.4 mm
- net OSC_IN: track 3.83 -> 5.25 mm
- added copper zone on layer 1, net 1.8V
- added copper zone on layer 1, net 5VIN
- added copper zone on layer 1, net 5VOUT
- added copper zone on layer 1, net GND
- added copper zone on layer 1, net N$7
- added copper zone on layer 1, net N$8
- added copper zone on layer 1, net VDD
