File: PCB/Team18_V1.3.brd (EAGLE design)
At the start: 98 x 100 mm, 63 parts, among them IC1 STM32F746ZGT6, J1 5.5x2.1mm Barrel, J2 CORTEX_DEBUG_PTH, P1 1-1473005-4, U1 TPPM0110DWPRDWP20_3P81X2P79-L, X1 2520-

Commit message: pcbsleep
Parts:
- removed HIGH_FREQ_OSC: 25 MHZ, SparkFun-Clocks:CRYSTAL-SMD-3.2X2.5MM
- added J3: 22-27-2041-04, con-molex:6410-04
- added Q1: (no value), adafruit:HC49UP
- moved J2 18.3 mm to (84.5, 95.6), turned to 0 degrees
- moved R3 10.9 mm to (47.5, 74.8), turned to 90 degrees
- moved C42 6.16 mm to (79.0, 95.4), flipped to the bottom, turned to 90 degrees
- moved C2 4.13 mm to (61.8, 57.9)
- moved C1 4.13 mm to (59.0, 57.9)
- moved LOW_FREQ_OSC 4.13 mm to (60.4, 58.9)
- moved R2 3.30 mm to (24.3, 66.7)
- moved P1 3.30 mm to (33.2, 47.5)
- moved C23 3.30 mm to (30.1, 76.6)
- moved C24 3.30 mm to (24.3, 76.6)
- moved C25 3.30 mm to (41.9, 76.6)
- moved C26 3.30 mm to (36.0, 76.6)
- moved C27 3.30 mm to (30.1, 81.5)
- moved C28 3.30 mm to (36.0, 81.5)
- moved C29 3.30 mm to (41.9, 81.5)
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Connections:
- new net SENSOR_UART: IC1.18, J3.2
- net GND: now also J3.4; no longer HIGH_FREQ_OSC.2, HIGH_FREQ_OSC.4
- net OSC_IN: now also Q1.1; no longer HIGH_FREQ_OSC.1
- net OSC_OUT: now also Q1.2; no longer HIGH_FREQ_OSC.3
- net VDD: now also J3.3
Routing:
- net GND: track 0.00 -> 278.3 mm, vias 0 -> 18
- net VDD: track 0.00 -> 115.3 mm, vias 0 -> 13
- net SWO: track 0.00 -> 57.7 mm
- net 5VOUT: track 0.00 -> 53.7 mm, vias 0 -> 1
- net QIO0: track 0.00 -> 42.1 mm
- net QIO2: track 0.00 -> 35.1 mm
- net 1.8V: track 0.00 -> 33.7 mm, vias 0 -> 1
- net QIO3: track 0.00 -> 31.9 mm
- net N$6: track 0.00 -> 31.2 mm, vias 0 -> 3
- net 5VIN: track 0.00 -> 23.3 mm
- net N$10: track 0.00 -> 21.9 mm, vias 0 -> 1
- net N$8: track 0.00 -> 19.7 mm
- net N$9: track 0.00 -> 17.0 mm, vias 0 -> 1
- net N$7: track 0.00 -> 12.7 mm
- net N$4: track 0.00 -> 12.3 mm, vias 0 -> 1
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