File: PCB/preauto.brd (EAGLE design)
At the start: 181.1 x 100 mm, 63 parts, among them IC1 STM32F746ZGT6, J1 5.5x2.1mm Barrel, P1 1-1473005-4, U1 TPPM0110DWPRDWP20_3P81X2P79-L, X1 2520-

Commit message: PCB
Parts:
- removed JTAG: (no value), Wurth_Elektronik_Electromechanic_Board_to_Board_Connectors_rev18b:62201021821
- added J2: CORTEX_DEBUG_PTH, SparkFun-Connectors:2X5-PTH-1.27MM
Connections:
- new net N$19: J2.8
- net 3.3V: no longer C23.1, C24.1, C25.1, C26.1, C35.1, C37.2, P1.191, P1.192, P1.193, P1.194, R3.2, U1.4
- net GND: now also J2.3, J2.5, J2.9; no longer JTAG.3, JTAG.5, JTAG.9
- net KEY: now also J2.7; no longer JTAG.7
- net RESET: now also J2.10; no longer IC1.134, JTAG.10
- net SWCLK: now also J2.4; no longer JTAG.4
- net SWDIO: now also J2.2; no longer JTAG.2
- net SWO: now also J2.6; no longer JTAG.6
- net VDD: now also C23.1, C24.1, C25.1, C26.1, C35.1, C37.2, J2.1, P1.191, P1.192, P1.193, P1.194, R3.2, U1.4; no longer JTAG.1
Routing:
- net 5VOUT: track 110.9 -> 265.4 mm, vias 3 -> 8
- net 3.3V: track 119.4 -> 27.3 mm, vias 2 -> 1
- net VDD: track 79.5 -> 140.4 mm, vias 15 -> 36
- net 5VIN: track 107.4 -> 70.5 mm
- net RESET: track 54.4 -> 77.1 mm
- net GND: track 533.2 -> 555.4 mm, vias 25 -> 46
- net N$6: track 19.6 -> 36.5 mm
- net RUN: track 0.00 -> 9.06 mm
- net N$1: track 0.00 -> 5.60 mm, vias 0 -> 1
- net 1.8V: track 47.1 -> 51.3 mm, vias 2 -> 10
- net OSC_OUT: track 5.74 -> 9.55 mm, vias 0 -> 1
- net N$8: track 18.5 -> 20.3 mm
- net QSPICLK: track 30.8 -> 32.4 mm
- net OSC32_IN: track 5.95 -> 7.54 mm
- net OSC_IN: track 6.74 -> 5.25 mm
- added copper zone on layer 1, net 1.8V
- added copper zone on layer 1, net 5VIN
- added copper zone on layer 1, net 5VOUT
- added copper zone on layer 1, net GND
- added copper zone on layer 1, net N$7
- added copper zone on layer 1, net N$8
- added copper zone on layer 1, net VDD
