File: PCB/MOSFETadded.brd (EAGLE design)
At the start: 100 x 100 mm, 68 parts, among them IC1 STM32F746ZGT6, J1 5.5x2.1mm Barrel, J2 CORTEX_DEBUG_PTH, P1 1-1473005-4, Q1 RZF013P01TL, Q2 RZF013P01TL, U1 TPPM0110DWPRDWP20_3P81X2P79-L, X2 USB-A

Commit message: prez
Routing:
- net 1.8V_PI: track 19.8 -> 18.7 mm
- net GND: vias 92 -> 99
Changed lines of the file:
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@@
 <vertex x="43.307" y="51.689"/>
 </polygon>
+<via x="41.148" y="56.007" extent="1-16" drill="0.3302"/>
+<via x="41.148" y="48.895" extent="1-16" drill="0.3302"/>
+<via x="41.148" y="40.64" extent="1-16" drill="0.3302"/>
+<via x="41.148" y="33.02" extent="1-16" drill="0.3302"/>
+<via x="48.133" y="59.817" extent="1-16" drill="0.3302"/>
+<via x="51.054" y="59.817" extent="1-16" drill="0.3302"/>
+<via x="48.26" y="56.261" extent="1-16" drill="0.3302"/>
+<wire x1="48.133" y1="59.817" x2="48.26" y2="56.261" width="0" layer="19" extent="1-1"/>
 </signal>
 <signal name="VDD">
@@
 <wire x1="39.624" y1="62.7415" x2="41.90999375" y2="62.7415" width="0.2032" layer="16"/>
 <via x="39.624" y="62.7415" extent="1-16" drill="0.3302" diameter="0.55"/>
-<wire x1="41.90999375" y1="61.59500625" x2="41.90999375" y2="62.7415" width="0.2032" layer="16"/>
 <polygon width="0.2032" layer="1">
 <vertex x="27.686" y="67.056"/>
