File: PCB/Presentation_PCB.brd (EAGLE design)
At the start: 100 x 100 mm, 68 parts, among them IC1 STM32F746ZGT6, J1 5.5x2.1mm Barrel, J2 CORTEX_DEBUG_PTH, P1 1-1473005-4, Q1 RZF013P01TL, Q2 RZF013P01TL, U1 TPPM0110DWPRDWP20_3P81X2P79-L, X2 USB-A

Commit message: prez
Routing:
- net QSPI_CS: track 44.8 -> 51.4 mm, vias 0 -> 2
- net SENSOR_UART: track 78.5 -> 76.7 mm
- net 1.8V_PI: track 19.8 -> 18.7 mm
- net D_P: track 54.5 -> 55.4 mm
- net D_N: track 55.4 -> 54.5 mm
- net GND: vias 92 -> 106
