File: PCB/Presentation_PCB.sch (EAGLE design)
At the start: 68 parts, among them IC1 STM32F746ZGT6, J1 5.5x2.1mm Barrel, J2 CORTEX_DEBUG_PTH, P1 1-1473005-4, U1 TPPM0110DWPRDWP20_3P81X2P79-L, U2 RQ5E035BNTCL, U3 RQ5E035BNTCL, U4 RQ5E035BNTCL, X2 USB-A

Commit message: prez
Parts:
- removed U2, U3, U4: RQ5E035BNTCL, 477_LIBRARY:RQ5E035BNTCL
- added Q1, Q2: RZF013P01TL, Pchannel:RZF013P01TL
Connections:
- removed net 5V_MOSFET: IC1.PE4, U4.G
- removed net N$11: U2.S
- removed net N$13: U2.D
- removed net N$14: U3.S
- removed net N$17: U3.D
- removed net N$18: U4.S
- removed net N$22: U4.D
- new net 1.8V_PI: C31.1, C32.1, C33.1, C34.1, P1.183, P1.184, P1.185, P1.186, Q2.D
- new net RUN_5V_MODULE: R10.1, U$1.RUN
- new net VDD_PI: C23.1, C24.1, C25.1, C26.1, P1.191, P1.192, P1.193, P1.194, Q1.D
- net 1.8V: now also Q2.S; no longer C31.1, C32.1, C33.1, C34.1, P1.183, P1.184, P1.185, P1.186
- net 1.8V_MOSFET: now also Q2.G; no longer U3.G
- net 5VOUT: no longer R10.2
- net RUN_5V: now also IC1.PE4, R10.2; no longer R10.1, U$1.RUN
- net VDD: now also Q1.S; no longer C23.1, C24.1, C25.1, C26.1, P1.191, P1.192, P1.193, P1.194
- net VDD_MOSFET: now also Q1.G; no longer U2.G
Other:
- note added: "5V Buck-Boost regulator"
- note added: "5V to 3.3V and 1.8V regulator"
- moved on the sheet: C18, C19, C20, C21, C22, C23, C24, C25, C26, C27, C28, C29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
