File: PCB/LoadSwitch.brd (EAGLE design)
At the start: 100 x 100 mm, 77 parts, among them IC1 STM32F746ZGT6, IC2 FPF2125, IC3 FPF2125, J1 5.5x2.1mm Barrel, J2 CORTEX_DEBUG_PTH, P1 1-1473005-4, U1 TPPM0110DWPRDWP20_3P81X2P79-L, X2 USB-A

Commit message: led
Parts:
- added D1, D2, D3, D4, D5, D6: (no value), SparkFun-LED:LED-0603
- added R16, R17, R18, R19, R20, R21: 1k, audio amplifier example:R0805
- moved R14 0.18 mm to (47.3, 55.4)
Connections:
- new net N$12: D6.C, R16.2
- new net N$13: D5.C, R17.2
- new net N$15: D1.C, R18.2
- new net N$16: D4.C, R19.2
- new net N$17: D3.C, R20.2
- new net N$18: D2.C, R21.2
- net 1.8V: now also D4.A
- net 1.8V_PI: now also D6.A
- net 5VIN: now also D1.A
- net 5VOUT: now also D2.A
- net GND: now also R16.1, R17.1, R18.1, R19.1, R20.1, R21.1
- net VDD: now also D3.A
- net VDD_PI: now also D5.A
Routing:
- net N$12: track 0.00 -> 2.94 mm
- net N$17: track 0.00 -> 2.54 mm
- net N$15: track 0.00 -> 2.25 mm
- net N$18: track 0.00 -> 2.21 mm
- net N$13: track 0.00 -> 2.12 mm
- net N$16: track 0.00 -> 2.07 mm
- net GND: track 352.5 -> 351.0 mm
Other:
- board text added: "1.8V LDO ON"
- board text added: "1.8V PI ON"
- board text added: "3.3V PI ON"
- board text added: "5V OUT ON"
- board text added: "Microcontroller ON"
- board text added: "Power ON"
- board text added: "Team 18: Parking Spot Finder Damini Rhijwani Noureldin Hendy Tania Chakraborty Richard Rao"
- board text added: "Two Things"
- board text removed: "PROXIMITY SENSOR"
